Commit message: feat(docking): 마커 3장 보드 기반 충전 도킹, 자동 복귀, 충전 중 절전
액션 규격은 Nav2 순정(/dock_robot, /undock_robot, opennav_docking 의
dock_database)을 그대로 쓴다. 실기 전환 시 도크 좌표만 바꾸면 되고 BT
연동도 살아 있다. 검출과 접근 방식만 자체 구현했다.

마커 3장을 하나의 보드로 푼다 (dock_marker_board.py)
  실물 스테이션에는 가이드 벽이 없어 최종 각도를 인식이 전적으로
  결정한다. 그런데 정면에 가까운 평면 마커 한 장은 자세 모호성 때문에
  1.3 m 에서 각도가 4.77도까지 튄다. 좌우 0.16 m 로 벌린 3장의 코너
  12개를 estimatePoseBoard 로 함께 풀면 같은 자리에서 0.01도 수준으로
  떨어진다. 세로로 쌓으면 yaw 개선 효과가 거의 없다 — 좌우 배치가 핵심.
  DICT_4X4_50 을 고른 이유는 424x240 해상도다. 테두리 포함 6칸이라
  24 px 이면 읽히지만 기본값 6x6 은 8칸이라 32 px 이 필요해 검출 거리가
  크게 짧아진다. 텍스처는 검출기와 같은 cv2 로 생성한다.

접근은 docking_mode 로 고른다 — 기본 staged, 비교용 smooth
  staged (staged_dock.py) 는 정지 -> 측정 -> 보정 -> 재측정을 반복한다.
  차동구동은 옆으로 못 가므로 횡오차는 크랩 기동으로 없앤다.
  실측 비교 (같은 월드/마커, 각 3~5회):
    세로 오차 중앙값/최대  staged 2.6/2.6 mm  vs  smooth 20.3/22.7 mm
    가로 오차              staged 1.2/5.5 mm  vs  smooth  0.8/ 2.4 mm
    각도 오차              staged 0.6/1.3도   vs  smooth  0.4/ 1.8도
    소요 시간 중앙값       staged 25.6초      vs  smooth  8.6초
  세로가 한 자릿수 이상 좋은 이유는 정지 상태 인식 정확도를 그대로 최종
  자세로 가져가기 때문이다. 곡선 접근은 그 측정값을 움직이면서 소비한다.

정렬 완료 판정은 축별 허용치가 아니라 "접촉 시점의 예상 횡오차" 하나
  횡오차와 각도오차는 독립이 아니다. 정렬 후 직진하는 동안 남은 각도가
  그대로 횡오차로 바뀐다:
      접촉 시점 횡오차 = 정렬시 횡오차 - 직진거리 x sin(각도오차)
  0.52 m 직진 기준 0.5도가 4.5 mm 다. 그래서 예전 설정(횡 3 mm /
  각도 0.5도)은 서로 앞뒤가 안 맞았다 — 허용한 각도만으로 4.5 mm 가
  생기는데 그보다 작은 3 mm 를 맞추려고 크랩을 반복했다(회당 15~20초
  손해). 지금은 contact_lateral_budget 하나로 판정하고 크랩 보정량도
  이 예상값을 쓴다. 예측 검증(예상 -> Gazebo 실제):
  +10.4 -> +5.5 mm, +0.9 -> +0.9 mm, +0.1 -> +1.2 mm.

충전 중에는 인지·항법을 재운다 (auto_dock.py, power_save)
  죽이지 말고 멈춰야 한다. rtabmap 을 죽였다 살리면 DB 를 다시 읽고
  재위치추정을 하는데 localization 모드는 오히려 CPU/메모리를 더 쓴다.
  /rtabmap/pause 는 포즈 그래프를 램에 둔 채 연산만 멈춘다.
  해제 순서가 중요하다: SLAM resume -> Nav2 RESUME -> 전역 코스트맵이
  실제로 다시 나오는 것을 확인 -> 그 다음에 언도킹. RESUME 완료와
  코스트맵 복귀 사이에 1.6초가 있고 그 사이 목표는 즉시 ABORT 된다.

도크 기하 — 접점 높이가 가장 빡빡한 제약
  동판 75x100 mm (실물 규격), 커넥터 6핀 2x3 피치 2.54 mm male DIP x2.
  전기적으로 닿아야 하는 면적은 핀 배열 6.1x3.5 mm 뿐이므로 접촉
  허용치는 (동판 - 핀 배열)/2 로 세로 +-48 mm / 가로 +-34 mm 다.
  30 mm 브래킷을 접촉면으로 잡으면 있지도 않은 정렬 정확도를 요구하게
  된다. 브래킷은 코스트맵 min_obstacle_height(0.030)와 접지고(0.060)
  사이에만 놓을 수 있어 0.045 m 다. 마커 높이는 화각 계산상 0.31 m —
  낮추면 근거리에서 화면 아래로 잘린다.

실측으로 드러난 함정 (전부 "로그는 멀쩡한데 안 되는" 부류)
- docking_server 의 enable_stamped_cmd_vel 기본값이 false 다. 그대로
  두면 Twist 를 내보내고 diff_drive_controller 가 조용히 무시한다.
- 접점 접촉 판정에 SLAM 자세를 쓰면 안 된다. 접근 루프는 isCharging()
  으로도 빠져나오므로 100 mm 앞에서 접근이 끝난다. 물리적 사실이므로
  Gazebo 지상 진실로 판정한다. 그래서 use_battery_status: false 로 두고
  충전 확인은 auto_dock 이 /battery_state 로 따로 한다.
- 좁은 가이드 벽 안에서는 코스트맵 충돌 검사가 원리적으로 동작하지
  않는다. 로봇 내접 반경의 2배보다 좁은 통로는 전체가
  INSCRIBED_INFLATED_OBSTACLE 로 칠해진다.
- 자세를 고정할 때 영상 타임스탬프로 TF 를 조회하면 미래 외삽으로 매번
  실패한다. timeout 을 줘도 소용없다 — 그 콜백이 단일 스레드 실행기를
  잡고 있어 TF 리스너 콜백이 돌 수 없다. 가장 최근 TF(stamp=0)로 조회.
- 멀티스레드 실행기에서 상태 기계는 잠가야 한다. 절전 해제가 수 초
  블록하는 사이 1 Hz 타이머가 다시 들어와 UndockRobot 이 4번 발행됐다.

frontier_explorer 에 /exploration_enabled 스위치를 넣었다. 충전 복귀는
DockRobot 이 내부적으로 NavigateToPose 를 거는데, 탐사가 2초마다 새
목표를 계속 보내면 그 이동을 밀어내 로봇이 도크로 가지 못한다.
nav2_startup_watchdog 은 감시 대상 lifecycle_manager 를 파라미터로
받게 했다 — 도킹 서버용 관리자에도 같은 증상이 난다.

측정 도구: tools/dock_calib.py (인식 정확도), dock_range.py (검출
범위·편차), dock_test.py (반복 도킹 성공률·정렬 오차).

Co-Authored-By: Claude Opus 5 (1M context) <noreply@anthropic.com>
Claude-Session: https://claude.ai/code/session_01WPh5dwdxzQ4cbRHgztAUdX

File: src/orinbot_description/urdf/orinbot.urdf.xacro (robot description, xacro)
@@ -40,4 +40,5 @@
   <material name="wheel_black"><color rgba="0.1 0.1 0.1 1.0"/></material>
   <material name="caster_silver"><color rgba="0.7 0.7 0.7 1.0"/></material>
+  <material name="pogo_gold"><color rgba="0.85 0.7 0.25 1.0"/></material>
   <!-- ======================= 본체 ======================= -->
   <!-- 지면에 투영된 기준 프레임 (Nav2 등이 사용) -->
@@ -61,4 +62,55 @@
       <origin xyz="0 0 0" rpy="0 0 0"/>
     </xacro:inertial_box>
+    <!-- 충전 포고핀 브래킷 (배면 좌우 2개, 각 6핀)
+      도크 바닥의 동판 위에 얹혀 접촉합니다.
+      높이가 이 로봇에서 가장 빡빡한 치수입니다.
+        섀시 바닥      0.060 m  (= 접지고. 캐스터 지름)
+        브래킷 하단    0.045 m  <- 여기
+        동판 상면      0.040 m  (generate_room.py 의 DOCK_PLATE_Z)
+                       =====
+        포고 스트로크  0.005 m
+      **0.030 m 아래로 내리면 안 됩니다.** 코스트맵의
+      min_obstacle_height 가 0.03 이라 로봇은 30 mm 미만 물체를 장애물로
+      보지 않고 그냥 밟고 지나갑니다 (월드의 3 cm 문턱이 그 경계 시험용).
+      브래킷이 그보다 낮으면 코스트맵이 무시한 물체에 그대로 걸립니다.
+      반대로 0.060 m 위로 올리면 섀시 안에 들어가 동판에 닿지 않습니다.
+      좌우 위치도 자유롭지 않습니다. 구동륜이 ±0.17, 캐스터가 ±0.14 에
+      있어 바퀴가 지나가지 않는 띠는 |y| < 0.11 뿐입니다. 동판이 바퀴
+      경로에 걸리면 로봇이 동판 위로 올라타 버려 브래킷과의 간격이
+      그대로 유지됩니다.
+    -->
+    <!--
+      실물 커넥터: 6핀 2x3 배열 / 피치 2.54 mm / male / DIP(관통홀) 2개.
+      아래 30 mm 각 상자는 그 커넥터와 기판을 붙드는 **브래킷**이지
+      접촉면이 아닙니다. 전기적으로 닿아야 하는 면적은 핀 배열
+      6.1 x 3.5 mm 뿐이고, 접촉 허용치는 거기서 나옵니다
+      (generate_room.py 가 계산해 찍어 줍니다: 세로 ±48, 가로 ±34 mm).
+      브래킷이 동판 밖으로 걸쳐 있어도 무방합니다.
+      실기 확인 필요: 동판 상면 40 mm, 브래킷 하단 45 mm 이므로 핀이
+      브래킷 아래로 5 mm 이상 나와 있어야 합니다. 2.54 mm 피치 포고핀의
+      스트로크는 보통 1.5~2.5 mm 라 **자유 길이로 5 mm 를 메우고 남는
+      만큼만 압축 여유**가 됩니다. 그 여유가 곧 바닥 높이 편차(램프
+      기울기, 동판 두께 공차) 허용치이므로 부품 데이터시트로 확인하세요.
+    -->
+    <xacro:property name="pogo_x" value="-0.10"/>      <!-- 배면 쪽 -->
+    <xacro:property name="pogo_y" value="0.055"/>
+    <xacro:property name="pogo_bottom" value="0.045"/>  <!-- 지면 기준 -->
+    <xacro:property name="pogo_size" value="0.03"/>     <!-- 브래킷, 접촉면 아님 -->
+    <xacro:property name="pogo_h" value="0.015"/>
+    <xacro:macro name="pogo_block" params="reflect">
+      <visual>
+        <origin xyz="${pogo_x} ${reflect * pogo_y}
+                     ${pogo_bottom + pogo_h/2.0 - base_z}" rpy="0 0 0"/>
+        <geometry><box size="${pogo_size} ${pogo_size} ${pogo_h}"/></geometry>
+        <material name="pogo_gold"/>
+      </visual>
+      <collision>
+        <origin xyz="${pogo_x} ${reflect * pogo_y}
+                     ${pogo_bottom + pogo_h/2.0 - base_z}" rpy="0 0 0"/>
+        <geometry><box size="${pogo_size} ${pogo_size} ${pogo_h}"/></geometry>
+      </collision>
+    </xacro:macro>
+    <xacro:pogo_block reflect="1"/>
+    <xacro:pogo_block reflect="-1"/>
   </link>
   <!-- ======================= 구동륜 ======================= -->
@@ -189,4 +241,30 @@
     <material>Gazebo/Grey</material>
   </gazebo>
+  <!-- ======================= 지상 진실 자세 (시뮬 전용) ======================= -->
+  <!--
+    Gazebo 가 아는 로봇의 "진짜" 자세를 내보냅니다. 실기에는 없는 것이므로
+    자율주행 스택은 절대 구독하면 안 됩니다. 쓰는 곳은 두 군데뿐입니다.
+      - battery_sim.py : 충전 접점이 실제로 맞닿았는지 판정
+      - tools/*.py     : SLAM 오차 측정의 기준값
+    왜 /world/room/dynamic_pose/info 를 브리지하지 않는가:
+    그 메시지에는 프레임 이름을 담는 header.data 가 없어서
+    ros_gz_bridge 의 Pose_V -> TFMessage 변환이 frame_id 를 전부 빈
+    문자열로 채웁니다. 그러면 어느 것이 로봇인지 구분할 수 없습니다
+    (실측 확인). OdometryPublisher 는 nav_msgs/Odometry 로 바로 나옵니다.
+    TF 는 내보내지 않습니다 — EKF 가 이미 odom->base_footprint 를
+    발행하고 있어 중복 발행이 되면 좌표계가 꼬입니다.
+  -->
+  <xacro:if value="$(arg sim_mode)">
+    <gazebo>
+      <plugin filename="gz-sim-odometry-publisher-system"
+              name="gz::sim::systems::OdometryPublisher">
+        <odom_frame>world</odom_frame>
+        <robot_base_frame>base_footprint</robot_base_frame>
+        <odom_topic>ground_truth/odom</odom_topic>
+        <odom_publish_frequency>20</odom_publish_frequency>
+        <dimensions>2</dimensions>
+      </plugin>
+    </gazebo>
+  </xacro:if>
   <!-- ======================= ros2_control ======================= -->
   <xacro:orinbot_ros2_control
